Commit message: husky_description : added support for simulating velodyne VLP-16 and HDL-32E sensors

File: husky_description/urdf/husky.urdf.xacro (robot description, xacro)
@@ -30,4 +30,9 @@
   <xacro:arg name="robot_namespace" default="/" />
   <xacro:arg name="urdf_extras" default="empty.urdf" />
+  <xacro:arg name="sensor_arch_enabled" default="true"/>
+  <xacro:arg name="sensor_arch_size" default="510"/>  <!-- 300, 510 -->
+  <xacro:arg name="velodyne_enabled" default="true"/>
+  <xacro:arg name="velodyne_model" default="vlp16"/>  <!-- vlp16, hdl32e -->
+  <xacro:arg name="velodyne_parent_link_name" default="sensor_arch_mount_link"/>
   <!-- Included URDF/XACRO Files -->
   <xacro:include filename="$(find husky_description)/urdf/decorations.urdf.xacro" />
@@ -36,4 +41,7 @@
   <xacro:include filename="$(find husky_description)/urdf/accessories/sick_lms1xx_mount.urdf.xacro"/>
   <xacro:include filename="$(find husky_description)/urdf/accessories/sensor_arch.urdf.xacro"/>
+  <xacro:include filename="$(find velodyne_description)/urdf/VLP-16.urdf.xacro"/>
+  <xacro:include filename="$(find velodyne_description)/urdf/HDL-32E.urdf.xacro"/>
+  <xacro:include filename="$(find ur_description)/urdf/ur5.urdf.xacro"/>
   <xacro:property name="M_PI" value="3.14159"/>
   <!-- Base Size -->
@@ -122,8 +130,21 @@
     </joint>
   </xacro:if>
+  <xacro:if value="$(arg sensor_arch_enabled)">
+    <xacro:property name="xacro_sensor_arch_size" value="$(arg sensor_arch_size)"/>
+    <xacro:sensor_arch prefix="" parent="top_plate_link" size="$(arg sensor_arch_size)">
+      <xacro:if value="${xacro_sensor_arch_size == 300}">
+	<origin xyz="-0.35 0 0.3" rpy="0 0 -3.14"/>
+      </xacro:if>
+      <xacro:if value="${xacro_sensor_arch_size != 300}">
+	<origin xyz="-0.35 0 0.51" rpy="0 0 -3.14"/>
+      </xacro:if>
+    </xacro:sensor_arch>
+  </xacro:if>
   <xacro:if value="$(arg kinect_enabled)">
+    <!--
     <xacro:sensor_arch prefix="" parent="top_plate_link">
       <origin xyz="-0.35 0 0.51" rpy="0 0 -3.14"/>
-    </xacro:sensor_arch>
+      </xacro:sensor_arch>
+      -->
     <joint name="kinect_frame_joint" type="fixed">
       <origin xyz="$(arg kinect_xyz)" rpy="$(arg kinect_rpy)" />

Commit message: husky_description: Added ur5_arm with modified mass and the hokuyo lidar

File: husky_description/urdf/husky.urdf.xacro (robot description, xacro)
@@ -1,38 +1,13 @@
 <?xml version="1.0"?>
-<!--
-Software License Agreement (BSD)
-\file      husky.urdf.xacro
-\authors   Paul Bovbel <pbovbel@clearpathrobotics.com>, Devon Ash <dash@clearpathrobotics.com>
-\copyright Copyright (c) 2015, Clearpath Robotics, Inc., All rights reserved.
-Redistribution and use in source and binary forms, with or without modification, are permitted provided that
-the following conditions are met:
- * Redistributions of source code must retain the above copyright notice, this list of conditions and the
-   following disclaimer.
- * Redistributions in binary form must reproduce the above copyright notice, this list of conditions and the
-   following disclaimer in the documentation and/or other materials provided with the distribution.
- * Neither the name of Clearpath Robotics nor the names of its contributors may be used to endorse or promote
-   products derived from this software without specific prior written permission.
-THIS SOFTWARE IS PROVIDED BY THE COPYRIGHT HOLDERS AND CONTRIBUTORS "AS IS" AND ANY EXPRESS OR IMPLIED WAR-
-RANTIES, INCLUDING, BUT NOT LIMITED TO, THE IMPLIED WARRANTIES OF MERCHANTABILITY AND FITNESS FOR A PARTICULAR
-PURPOSE ARE DISCLAIMED. IN NO EVENT SHALL THE COPYRIGHT HOLDER OR CONTRIBUTORS BE LIABLE FOR ANY DIRECT, IN-
-DIRECT, INCIDENTAL, SPECIAL, EXEMPLARY, OR CONSEQUENTIAL DAMAGES (INCLUDING, BUT NOT LIMITED TO, PROCUREMENT
-OF SUBSTITUTE GOODS OR SERVICES; LOSS OF USE, DATA, OR PROFITS; OR BUSINESS INTERRUPTION) HOWEVER CAUSED AND
-ON ANY THEORY OF LIABILITY, WHETHER IN CONTRACT, STRICT LIABILITY, OR TORT (INCLUDING NEGLIGENCE OR OTHERWISE)
-ARISING IN ANY WAY OUT OF THE USE OF THIS SOFTWARE, EVEN IF ADVISED OF THE POSSIBILITY OF SUCH DAMAGE.
--->
 <robot name="husky" xmlns:xacro="http://ros.org/wiki/xacro">
   <xacro:arg name="laser_enabled" default="false" />
-  <xacro:arg name="laser_xyz" default="$(optenv HUSKY_LMS1XX_XYZ 0.2206 0.0 0.00635)" />
+  <xacro:arg name="laser_xyz" default="$(optenv HUSKY_LMS1XX_XYZ 0.4 0.0 -0.3)" />
   <xacro:arg name="laser_rpy" default="$(optenv HUSKY_LMS1XX_RPY 0.0 0.0 0.0)" />
+  <xacro:arg name="velodyne_enabled" default="true"/>
+  <xacro:arg name="ur5_enabled" default="true"/>
   <xacro:arg name="kinect_enabled" default="false" />
   <xacro:arg name="kinect_xyz" default="$(optenv HUSKY_KINECT_XYZ 0 0 0)" />
   <xacro:arg name="kinect_rpy" default="$(optenv HUSKY_KINECT_RPY 0 0.18 3.14)" />
-  <xacro:arg name="robot_namespace" default="/" />
   <xacro:arg name="urdf_extras" default="empty.urdf" />
-  <xacro:arg name="sensor_arch_enabled" default="true"/>
-  <xacro:arg name="sensor_arch_size" default="510"/>  <!-- 300, 510 -->
-  <xacro:arg name="velodyne_enabled" default="true"/>
-  <xacro:arg name="velodyne_model" default="vlp16"/>  <!-- vlp16, hdl32e -->
-  <xacro:arg name="velodyne_parent_link_name" default="sensor_arch_mount_link"/>
   <!-- Included URDF/XACRO Files -->
   <xacro:include filename="$(find husky_description)/urdf/decorations.urdf.xacro" />
@@ -40,8 +15,8 @@
   <xacro:include filename="$(find husky_description)/urdf/accessories/kinect_camera.urdf.xacro"/>
   <xacro:include filename="$(find husky_description)/urdf/accessories/sick_lms1xx_mount.urdf.xacro"/>
+  <xacro:include filename="$(find husky_description)/urdf/accessories/hokuyo.urdf.xacro"/>
   <xacro:include filename="$(find husky_description)/urdf/accessories/sensor_arch.urdf.xacro"/>
   <xacro:include filename="$(find velodyne_description)/urdf/VLP-16.urdf.xacro"/>
-  <xacro:include filename="$(find velodyne_description)/urdf/HDL-32E.urdf.xacro"/>
-  <xacro:include filename="$(find ur_description)/urdf/ur5.urdf.xacro"/>
+  <xacro:include filename="$(find husky_description)/urdf/accessories/ur5.urdf.xacro"/>
   <xacro:property name="M_PI" value="3.14159"/>
   <!-- Base Size -->
@@ -122,5 +97,5 @@
   <xacro:husky_decorate />
   <xacro:if value="$(arg laser_enabled)">
-    <sick_lms1xx_mount prefix="base"/>
+    <!--sick_lms1xx_mount prefix="base"/>
     <sick_lms1xx frame="base_laser" topic="scan" robot_namespace="$(arg robot_namespace)"/>
     <joint name="laser_mount_joint" type="fixed">
@@ -128,23 +103,47 @@
       <parent link="top_plate_link" />
       <child link="base_laser_mount" />
-    </joint>
+    </joint-->
+    <hokuyo_laser xyz="$(arg laser_xyz)" rpy="$(arg laser_rpy)" parent="top_plate_link"/>
   </xacro:if>
-  <xacro:if value="$(arg sensor_arch_enabled)">
-    <xacro:property name="xacro_sensor_arch_size" value="$(arg sensor_arch_size)"/>
-    <xacro:sensor_arch prefix="" parent="top_plate_link" size="$(arg sensor_arch_size)">
-      <xacro:if value="${xacro_sensor_arch_size == 300}">
-	<origin xyz="-0.35 0 0.3" rpy="0 0 -3.14"/>
-      </xacro:if>
-      <xacro:if value="${xacro_sensor_arch_size != 300}">
-	<origin xyz="-0.35 0 0.51" rpy="0 0 -3.14"/>
-      </xacro:if>
-    </xacro:sensor_arch>
+  <xacro:if value="$(arg ur5_enabled)">
+      <xacro:property name="reflect" value="-1" />
+      <!-- Spawn arm -->
+      <xacro:ur5_robot prefix="ur5_arm_" joint_limited="true"/>
+      <!-- Join arm -->
+      <joint name="ur5_arm_base" type="fixed">
+        <parent link="top_plate_link" />
+        <child link="ur5_arm_base_link" />
+        <origin xyz="0.3058 0 0.0065" rpy="0.0 0.0 -1.57" />
+      </joint>
+      <!--Remove when https://github.com/ros-industrial/universal_robot/pull/168 is resolved -->
+      <!--gazebo reference="ur5_arm_shoulder_link">
+        <selfCollide>true</selfCollide>
+      </gazebo>
+      <gazebo reference="ur5_arm_upper_arm_link">
+        <selfCollide>true</selfCollide>
+      </gazebo>
+      <gazebo reference="ur5_arm_forearm_link">
+        <selfCollide>true</selfCollide>
+      </gazebo>
+      <gazebo reference="ur5_arm_wrist_1_link">
+        <selfCollide>true</selfCollide>
+      </gazebo>
+      <gazebo reference="ur5_arm_wrist_3_link">
+       <selfCollide>true</selfCollide>
+      </gazebo>
+      <gazebo reference="ur5_arm_wrist_2_link">
+        <selfCollide>true</selfCollide>
+      </gazebo>
+      <gazebo reference="ur5_arm_ee_link">
+        <selfCollide>true</selfCollide>
+      </gazebo-->
+    </xacro:if>
+  <xacro:sensor_arch prefix="" parent="top_plate_link" size="300">
+      <origin xyz="-0.35 0 0.30" rpy="0 0 -3.14"/>
+  </xacro:sensor_arch>
+  <xacro:if value="$(arg velodyne_enabled)">
+     <xacro:VLP-16 parent="sensor_arch_mount_link"/>
   </xacro:if>
   <xacro:if value="$(arg kinect_enabled)">
-    <!--
-    <xacro:sensor_arch prefix="" parent="top_plate_link">
-      <origin xyz="-0.35 0 0.51" rpy="0 0 -3.14"/>
-      </xacro:sensor_arch>
-      -->
     <joint name="kinect_frame_joint" type="fixed">
       <origin xyz="$(arg kinect_xyz)" rpy="$(arg kinect_rpy)" />
