Commit message: move_base: Integrated the move_base function and static playpen map to the simulation

File: husky_description/urdf/accessories/hokuyo.urdf.xacro (robot description, xacro)
@@ -36,13 +36,13 @@
                 <scan>
                     <horizontal>
-                        <samples>360</samples>
+                        <samples>100</samples>
                         <resolution>1</resolution>
-                        <min_angle>-3.14159/2</min_angle>
-                        <max_angle>3.14159/2</max_angle>
+                        <min_angle>-1.0</min_angle>
+                        <max_angle>1.0</max_angle>
                     </horizontal>
                 </scan>
                 <range>
-                    <min>0.2</min>
-                    <max>40</max>
+                    <min>0.3</min>
+                    <max>5</max>
                     <resolution>0.025</resolution>
                 </range>
@@ -55,5 +55,5 @@
             <plugin name="gazebo_ros_head_hokuyo_controller" filename="libgazebo_ros_laser.so">
                 <robotNamespace></robotNamespace>
-                <topicName>laser_scan</topicName>
+                <topicName>scan</topicName>
                 <frameName>hokuyo_laser_link</frameName>
             </plugin>

File: husky_description/urdf/accessories/ur5.urdf.xacro (robot description, xacro)
@@ -102,5 +102,5 @@
       <parent link="${prefix}base_link" />
       <child link = "${prefix}shoulder_link" />
-      <origin xyz="0.0 0.0 ${shoulder_height}" rpy="0.0 0.0 ${pi}" /><!--z 0.0-->
+      <origin xyz="0.0 0.0 ${shoulder_height}" rpy="0.0 0.0 ${1.5 * pi}" /><!--z 0.0-->
       <axis xyz="0 0 1" />
       <xacro:unless value="${joint_limited}">

File: husky_description/urdf/husky.urdf.xacro (robot description, xacro)
@@ -9,4 +9,5 @@
   <xacro:arg name="kinect_xyz" default="$(optenv HUSKY_KINECT_XYZ 0 0 0)" />
   <xacro:arg name="kinect_rpy" default="$(optenv HUSKY_KINECT_RPY 0 0.18 3.14)" />
+  <xacro:arg name="robot_namespace" default="\"/>
   <xacro:arg name="urdf_extras" default="empty.urdf" />
   <!-- Included URDF/XACRO Files -->
